File: board/rev0.3/086-005.brd (EAGLE design)
At the start: 44.5 x 52.2 mm, 36 parts, among them IC1 MEGA48/88/168-AU, IC3 A4982, IC6 75176AD, IC8 TL780_VREG, J2 AVR-ISP-6VERT, J3 KK-4P, J9 22-27-2021-02, Q1 18.432MHz

Commit message: added an extra connector so you can use multiple cables for connecting
Parts:
- moved IC8 0.40 mm to (37.8, 16.6)
Routing:
- net GND: track 255.1 -> 305.1 mm, vias 29 -> 30
- net +24V: track 148.1 -> 141.8 mm
- net RS485-B: track 34.7 -> 32.6 mm, vias 2 -> 1
Other:
- board text added: "gestalt node"
- board text added: "rev 0.3, jun 2014"
